File: SWS600-12.kicad_sch (KiCad schematic)
At the start: 262 parts, among them CN1 OUT, CN2 CONTROL, CN3 TEMP, CN51 OUT, CN52 CONTROL, CN53 TEMP IN, CN54 FAN, Q1 2SK2837, Q100 2SK2177, Q101 "841"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

Commit message: update some part values, add images
Parts:
- added C205: 1uF, symbol Device:C_Small
- added E1, E2, E3, E4: SparkGap, symbol Device:SparkGap
- added Q203: NO STUFF, symbol Device:Q_NPN_BCE
- C10, C3, C4, C9: value ? -> 2.2nF
- C16: value ? -> 220pF
- C201, C217, C219, C220: value ? -> 10nF
- C202: value ? -> 4nF?
- C204: value ? -> 0.2uF?
- C206, C221: value ? -> 0.47uF
- C218: value ? -> 2.2uF
- C222: value ? -> 68nF?
- C223: value ? -> 5.5nF?
- C224: value ? -> 13nF?
- C225, C5, C6, C7: value ? -> 1uF
- L1: value ? -> 4.7mH
- L2: value ? -> 6.6mH
- L6: value ? -> 120uH
- SA1: value ? -> ERZV10D471
- renumbered C16 to C13, R217 to R252
Connections:
- net GNDD: now also C205.2, Q203.3 (E)
- net GNDS: now also R222.2
- net at PC54.4, R228.2, R230.1: now also Q203.1 (B)
- net at CN53.2 (Pin_2), D205.1 (K), R227.1: now also C205.1
- net at C1.1, C14.1, F1.2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: now also E1.1
- net at C2.2, C4.1, L1.4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: now also E2.2, E4.1
- net at C2.1, C3.2, L1.3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: now also E1.2, E3.1
- net at C14.2, L1.1, L6.2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: now also E2.1
- net at D1.2, L2.3, SA1.1: now also E3.2
- net at D1.3, L2.4, SA1.2: now also E4.2
- net at R228.1, R229.1, U200.7 (ON): now also Q203.2 (C)
Other:
- note added: "450V"
- note added: "470V"
- note added: "50W-4053"
- note added: "R228=0, Q203=DNI: ON/OFF=high for power up R228=DNI, Q203=npn: ON/OFF=low for power up (as in manual)"
- moved on the sheet: CN53, L1, R228, R229, R230, TS51
